Commit message: fix: preserve reviewed mesh material contracts

File: ros2_ws/src/ayyo_description/urdf/ayyo_geometry.xacro (robot description, xacro)
@@ -31,5 +31,7 @@
           </xacro:unless>
         </geometry>
-        <material name="${material}"/>
+        <xacro:unless value="${use_meshes}">
+          <material name="${material}"/>
+        </xacro:unless>
       </visual>
       <collision>
