Commit message: feat: activate Gazebo ros2 control hardware contract

File: ros2_ws/src/ayyo_description/urdf/ayyo.urdf.xacro (robot description, xacro)
@@ -4,4 +4,6 @@
   <xacro:arg name="simulation_mode" default="false"/>
   <xacro:arg name="simulation_static" default="true"/>
+  <xacro:arg name="simulation_control" default="false"/>
+  <xacro:arg name="simulation_controller_config" default=""/>
   <xacro:include filename="ayyo_materials.xacro"/>
   <xacro:include filename="ayyo_geometry.xacro"/>
@@ -12,5 +14,12 @@
   <xacro:ayyo_body use_meshes="$(arg use_meshes)"/>
   <xacro:if value="$(arg simulation_mode)">
-    <xacro:ayyo_gazebo static_model="$(arg simulation_static)"/>
+    <xacro:ayyo_gazebo
+      static_model="$(arg simulation_static)"
+      control_enabled="$(arg simulation_control)"
+      controller_config="$(arg simulation_controller_config)"/>
+    <xacro:if value="$(arg simulation_control)">
+      <xacro:ayyo_ros2_control_system
+        hardware_plugin="gz_ros2_control/GazeboSimSystem"/>
+    </xacro:if>
   </xacro:if>
 </robot>

File: ros2_ws/src/ayyo_description/urdf/ayyo_gazebo.xacro (robot description, xacro)
@@ -1,12 +1,17 @@
 <?xml version="1.0"?>
 <robot xmlns:xacro="http://www.ros.org/wiki/xacro">
-  <xacro:macro name="ayyo_gazebo" params="static_model">
-    <!--
-      Foundation v1 deliberately spawns a static, non-actuating development
-      model. No Gazebo system plugin, controller, or hardware interface is
-      loaded by the authoritative description.
-    -->
+  <xacro:macro name="ayyo_gazebo"
+               params="static_model control_enabled controller_config">
     <gazebo>
-      <static>${str(static_model).lower()}</static>
+      <xacro:if value="${control_enabled}">
+        <static>false</static>
+        <plugin filename="gz_ros2_control-system"
+                name="gz_ros2_control::GazeboSimROS2ControlPlugin">
+          <parameters>${controller_config}</parameters>
+        </plugin>
+      </xacro:if>
+      <xacro:unless value="${control_enabled}">
+        <static>${str(static_model).lower()}</static>
+      </xacro:unless>
     </gazebo>
   </xacro:macro>

File: ros2_ws/src/ayyo_description/urdf/ayyo_ros2_control.xacro (robot description, xacro)
@@ -1,15 +1,13 @@
 <?xml version="1.0"?>
 <robot xmlns:xacro="http://www.ros.org/wiki/xacro">
-  <!--
-    This macro is a dormant interface contract. Foundation v1 never invokes
-    it and supplies no hardware plugin. A later reviewed integration may call
-    it only after choosing a concrete simulation or hardware system below the
-    Runtime Bridge and physical-safety boundaries.
-  -->
-  <xacro:macro name="ayyo_controlled_joint" params="name">
+  <xacro:macro name="ayyo_ros2_control_joint" params="name command_position">
     <joint name="${name}">
-      <!-- Position limits remain single-owned by the corresponding URDF joint. -->
-      <command_interface name="position"/>
-      <state_interface name="position"/>
+      <xacro:if value="${command_position}">
+        <!-- Limits remain single-owned by the corresponding URDF joint. -->
+        <command_interface name="position"/>
+      </xacro:if>
+      <state_interface name="position">
+        <param name="initial_value">0.0</param>
+      </state_interface>
       <state_interface name="velocity"/>
       <state_interface name="effort"/>
@@ -21,22 +19,25 @@
         <plugin>${hardware_plugin}</plugin>
       </hardware>
-      <xacro:ayyo_controlled_joint name="neck_yaw_joint"/>
-      <xacro:ayyo_controlled_joint name="head_pitch_joint"/>
-      <xacro:ayyo_controlled_joint name="left_shoulder_yaw_joint"/>
-      <xacro:ayyo_controlled_joint name="left_shoulder_pitch_joint"/>
-      <xacro:ayyo_controlled_joint name="left_elbow_flex_joint"/>
-      <xacro:ayyo_controlled_joint name="left_wrist_yaw_joint"/>
-      <xacro:ayyo_controlled_joint name="right_shoulder_yaw_joint"/>
-      <xacro:ayyo_controlled_joint name="right_shoulder_pitch_joint"/>
-      <xacro:ayyo_controlled_joint name="right_elbow_flex_joint"/>
-      <xacro:ayyo_controlled_joint name="right_wrist_yaw_joint"/>
-      <xacro:ayyo_controlled_joint name="left_hip_yaw_joint"/>
-      <xacro:ayyo_controlled_joint name="left_hip_pitch_joint"/>
-      <xacro:ayyo_controlled_joint name="left_knee_flex_joint"/>
-      <xacro:ayyo_controlled_joint name="left_ankle_pitch_joint"/>
-      <xacro:ayyo_controlled_joint name="right_hip_yaw_joint"/>
-      <xacro:ayyo_controlled_joint name="right_hip_pitch_joint"/>
-      <xacro:ayyo_controlled_joint name="right_knee_flex_joint"/>
-      <xacro:ayyo_controlled_joint name="right_ankle_pitch_joint"/>
+      <!-- V1 intentionally exposes one and only one command interface. -->
+      <xacro:ayyo_ros2_control_joint
+        name="neck_yaw_joint" command_position="true"/>
+      <xacro:ayyo_ros2_control_joint
+        name="head_pitch_joint" command_position="false"/>
+      <xacro:ayyo_ros2_control_joint name="left_shoulder_yaw_joint" command_position="false"/>
+      <xacro:ayyo_ros2_control_joint name="left_shoulder_pitch_joint" command_position="false"/>
+      <xacro:ayyo_ros2_control_joint name="left_elbow_flex_joint" command_position="false"/>
+      <xacro:ayyo_ros2_control_joint name="left_wrist_yaw_joint" command_position="false"/>
+      <xacro:ayyo_ros2_control_joint name="right_shoulder_yaw_joint" command_position="false"/>
+      <xacro:ayyo_ros2_control_joint name="right_shoulder_pitch_joint" command_position="false"/>
+      <xacro:ayyo_ros2_control_joint name="right_elbow_flex_joint" command_position="false"/>
+      <xacro:ayyo_ros2_control_joint name="right_wrist_yaw_joint" command_position="false"/>
+      <xacro:ayyo_ros2_control_joint name="left_hip_yaw_joint" command_position="false"/>
+      <xacro:ayyo_ros2_control_joint name="left_hip_pitch_joint" command_position="false"/>
+      <xacro:ayyo_ros2_control_joint name="left_knee_flex_joint" command_position="false"/>
+      <xacro:ayyo_ros2_control_joint name="left_ankle_pitch_joint" command_position="false"/>
+      <xacro:ayyo_ros2_control_joint name="right_hip_yaw_joint" command_position="false"/>
+      <xacro:ayyo_ros2_control_joint name="right_hip_pitch_joint" command_position="false"/>
+      <xacro:ayyo_ros2_control_joint name="right_knee_flex_joint" command_position="false"/>
+      <xacro:ayyo_ros2_control_joint name="right_ankle_pitch_joint" command_position="false"/>
     </ros2_control>
   </xacro:macro>

Commit message: feat: add default-off Stage 9C controller profile

File: ros2_ws/src/ayyo_description/urdf/ayyo.urdf.xacro (robot description, xacro)
@@ -5,4 +5,5 @@
   <xacro:arg name="simulation_static" default="true"/>
   <xacro:arg name="simulation_control" default="false"/>
+  <xacro:arg name="simulation_manipulation_control" default="false"/>
   <xacro:arg name="simulation_localization" default="false"/>
   <xacro:arg name="simulation_camera" default="false"/>
@@ -26,5 +27,6 @@
     <xacro:if value="$(arg simulation_control)">
       <xacro:ayyo_ros2_control_system
-        hardware_plugin="gz_ros2_control/GazeboSimSystem"/>
+        hardware_plugin="gz_ros2_control/GazeboSimSystem"
+        manipulation_control="$(arg simulation_manipulation_control)"/>
     </xacro:if>
   </xacro:if>

File: ros2_ws/src/ayyo_description/urdf/ayyo_ros2_control.xacro (robot description, xacro)
@@ -1,5 +1,5 @@
 <?xml version="1.0"?>
 <robot xmlns:xacro="http://www.ros.org/wiki/xacro">
-  <xacro:macro name="ayyo_ros2_control_joint" params="name command_position">
+  <xacro:macro name="ayyo_ros2_control_joint" params="name command_position initial_value:=0.0">
     <joint name="${name}">
       <xacro:if value="${command_position}">
@@ -8,5 +8,5 @@
       </xacro:if>
       <state_interface name="position">
-        <param name="initial_value">0.0</param>
+        <param name="initial_value">${initial_value}</param>
       </state_interface>
       <state_interface name="velocity"/>
@@ -14,18 +14,19 @@
     </joint>
   </xacro:macro>
-  <xacro:macro name="ayyo_ros2_control_system" params="hardware_plugin">
+  <xacro:macro name="ayyo_ros2_control_system" params="hardware_plugin manipulation_control:=false">
     <ros2_control name="AyyoSystem" type="system">
       <hardware>
         <plugin>${hardware_plugin}</plugin>
       </hardware>
-      <!-- V1 intentionally exposes one and only one command interface. -->
+      <!-- The normal profile retains only the neck command. Stage 9C replaces
+           it with exactly four left-arm position commands when explicitly set. -->
       <xacro:ayyo_ros2_control_joint
-        name="neck_yaw_joint" command_position="true"/>
+        name="neck_yaw_joint" command_position="${not manipulation_control}"/>
       <xacro:ayyo_ros2_control_joint
         name="head_pitch_joint" command_position="false"/>
-      <xacro:ayyo_ros2_control_joint name="left_shoulder_yaw_joint" command_position="false"/>
-      <xacro:ayyo_ros2_control_joint name="left_shoulder_pitch_joint" command_position="false"/>
-      <xacro:ayyo_ros2_control_joint name="left_elbow_flex_joint" command_position="false"/>
-      <xacro:ayyo_ros2_control_joint name="left_wrist_yaw_joint" command_position="false"/>
+      <xacro:ayyo_ros2_control_joint name="left_shoulder_yaw_joint" command_position="${manipulation_control}"/>
+      <xacro:ayyo_ros2_control_joint name="left_shoulder_pitch_joint" command_position="${manipulation_control}"/>
+      <xacro:ayyo_ros2_control_joint name="left_elbow_flex_joint" command_position="${manipulation_control}" initial_value="${0.2 if manipulation_control else 0.0}"/>
+      <xacro:ayyo_ros2_control_joint name="left_wrist_yaw_joint" command_position="${manipulation_control}"/>
       <xacro:ayyo_ros2_control_joint name="right_shoulder_yaw_joint" command_position="false"/>
       <xacro:ayyo_ros2_control_joint name="right_shoulder_pitch_joint" command_position="false"/>

Commit message: fix: bind Stage 9C support and stability evidence

File: ros2_ws/src/ayyo_description/urdf/ayyo.urdf.xacro (robot description, xacro)
@@ -6,4 +6,5 @@
   <xacro:arg name="simulation_control" default="false"/>
   <xacro:arg name="simulation_manipulation_control" default="false"/>
+  <xacro:arg name="simulation_manipulation_support" default="false"/>
   <xacro:arg name="simulation_localization" default="false"/>
   <xacro:arg name="simulation_camera" default="false"/>
@@ -25,5 +26,6 @@
       depth_camera_enabled="$(arg simulation_depth_camera)"
       controller_config="$(arg simulation_controller_config)"
-      manipulation_control_enabled="$(arg simulation_manipulation_control)"/>
+      manipulation_control_enabled="$(arg simulation_manipulation_control)"
+      manipulation_support_enabled="$(arg simulation_manipulation_support)"/>
     <xacro:if value="$(arg simulation_control)">
       <xacro:ayyo_ros2_control_system

File: ros2_ws/src/ayyo_description/urdf/ayyo_gazebo.xacro (robot description, xacro)
@@ -2,14 +2,17 @@
 <robot xmlns:xacro="http://www.ros.org/wiki/xacro">
   <xacro:macro name="ayyo_gazebo"
-               params="static_model control_enabled localization_enabled camera_enabled depth_camera_enabled controller_config manipulation_control_enabled">
+               params="static_model control_enabled localization_enabled camera_enabled depth_camera_enabled controller_config manipulation_control_enabled manipulation_support_enabled">
     <xacro:if value="${control_enabled}">
       <xacro:if value="${manipulation_control_enabled}">
-        <!-- Stage 9C uses gravity-neutral development dynamics for the arm.
-             This opt-in has no physical-controller or validation meaning. -->
-        <gazebo reference="left_upper_arm_link"><gravity>false</gravity></gazebo>
-        <gazebo reference="left_elbow_link"><gravity>false</gravity></gazebo>
-        <gazebo reference="left_forearm_link"><gravity>false</gravity></gazebo>
-        <gazebo reference="left_wrist_link"><gravity>false</gravity></gazebo>
-        <gazebo reference="left_hand_link"><gravity>false</gravity></gazebo>
+        <xacro:if value="${manipulation_support_enabled}">
+          <!-- Explicit simulation-only Stage 9C manipulation fixture. The
+               articulated model remains dynamic and collisions/gravity remain
+               enabled; only its free base is anchored for this bounded proof. -->
+          <link name="world"/>
+          <joint name="stage9c_manipulation_fixture_joint" type="fixed">
+            <parent link="world"/>
+            <child link="base_link"/>
+          </joint>
+        </xacro:if>
       </xacro:if>
     </xacro:if>
